Commit message: integrate relative motion and odometry calibration

File: src/agv_description/urdf/agv.urdf.xacro (robot description, xacro)
@@ -29,5 +29,5 @@
     <parent link="base_link"/>
     <child link="laser_frame"/>
-    <origin xyz="0.230 0.0 0.255" rpy="0.0 0.0 0.0"/>
+    <origin xyz="-0.230 0.0 0.255" rpy="0.0 0.0 0.0"/>
   </joint>
   <link name="laser_frame">

Commit message: Finalize AGV navigation workspace

File: src/agv_description/urdf/agv.urdf.xacro (robot description, xacro)
@@ -29,5 +29,5 @@
     <parent link="base_link"/>
     <child link="laser_frame"/>
-    <origin xyz="-0.230 0.0 0.255" rpy="0.0 0.0 0.0"/>
+    <origin xyz="0.120 0.0 0.255" rpy="0.0 0.0 3.141592653589793"/>
   </joint>
   <link name="laser_frame">
